File: _autosave-pwr_clk.kicad_sch (KiCad schematic)
At the start: 3 parts, among them J3 Conn_01x02_Pin, U4 LM1117DT-3.3

Commit message: connector update
Connections:
- net 3V3: now reaches U4.2 (VO)
Other:
- note added: "Regülatör U4 - LM1117DT-3.3 Giriş: SYS_UPS (5-9 V arası) Çıkış: +3.3 V nominal Max Iout: ~800 mA Giriş/Çıkış farkı yüksek olduğunda termal kayıplar artar. Gerekirse buck regülatör alternatifi değerlendirilecektir."
Changed lines of the file:
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@@
 	(generator_version "9.0")
 	(paper "A4")
+	(text "Regülatör U4 - LM1117DT-3.3\nGiriş: SYS_UPS (5-9 V arası)\nÇıkış: +3.3 V nominal\nMax Iout: ~800 mA\nGiriş/Çıkış farkı yüksek olduğunda termal kayıplar artar.\nGerekirse buck regülatör alternatifi değerlendirilecektir.\n"
+		(exclude_from_sim no)
+		(at 57.404 17.526 0)
+		(effects
+			(font
+				(size 0.7 0.7)
+			)
+		)
+	)
 	(junction
 		(at 30.48 29.21)
@@
 		(effects
 			(font
+				(size 0.7 0.7)
+			)
+			(justify left bottom)
+		)
+	)
+	(label "3V3"
+		(at 53.34 29.21 0)
+		(effects
+			(font
+				(size 0.7 0.7)
+			)
+			(justify left bottom)
+		)
+	)
+	(label "SYS_UPS"
+		(at 34.29 29.21 0)
+		(effects
+			(font
