File: pwr_clk.kicad_sch (KiCad schematic)
At the start: 0 parts

Commit message: connector update
Parts:
- added C3: 10 µF, symbol Device:C_Small
- added J3: Conn_01x02_Pin, symbol Connector:Conn_01x02_Pin
- added U4: LM1117DT-3.3, Package_TO_SOT_SMD:TO-252-3_TabPin2, symbol Regulator_Linear:LM1117DT-3.3
Connections:
- new net +5V_IN: C3.2, J3.1 (Pin_1), U4.3 (VI)
- new net GND: C3.1, J3.2 (Pin_2)

Commit message: usb-c add and save
Parts:
- added C4, C6: 100 nF, symbol Device:C_Small
- added C5, C7: 10 µF, symbol Device:C_Small
- added FB3: FerriteBead_Small, symbol Device:FerriteBead_Small
- added J4: USB_C_Receptacle_USB2.0_16P, symbol Connector:USB_C_Receptacle_USB2.0_16P
Connections:
- net GND: now also U4.1 (GND), C4.2, C5.2, C6.1, C7.1
- net 3V3: now reaches U4.2 (VO)
- net 3V3: now also C4.1, C5.1, FB3.1
- new net: J4.A1 (GND), J4.A12 (GND), J4.B1 (GND), J4.B12 (GND)
- new net: J4.A4 (VBUS), J4.A9 (VBUS), J4.B4 (VBUS), J4.B9 (VBUS)
- new net 3v3_RF: C6.2, C7.2, FB3.2
Other:
- note added: "Regülatör U4 - LM1117DT-3.3 Giriş: SYS_UPS (5-9 V arası) Çıkış: +3.3 V nominal Max Iout: ~800 mA Giriş/Çıkış farkı yüksek olduğunda termal kayıplar artar. Gerekirse buck regülatör alternatifi değerlendirilecektir."
- moved on the sheet: C3, J3, U4

Commit message: sync
Parts:
- removed J3: Conn_01x02_Pin, symbol Connector:Conn_01x02_Pin
- added D2, D3: D_Schottky, symbol Device:D_Schottky
Connections:
- net +5V_IN: now also D2.2 (A)
- net 5V_USB: now reaches J4.A4 (VBUS), J4.A9 (VBUS), J4.B4 (VBUS), J4.B9 (VBUS)
- net 5V_USB: now also D2.1 (K)
Other:
- moved on the sheet: J4
Changed lines of the file:
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@@
-	)
-	(junction
-		(at 67.31 30.48)
-		(diameter 0)
-		(color 0 0 0 0)
 	)
 	(junction
@@
 	(wire
 		(pts
-			(xy 67.31 30.48) (xy 72.39 30.48)
-		)
-		(stroke
-			(width 0)
-			(type default)
-		)
-	)
-	(wire
-		(pts
 			(xy 72.39 30.48) (xy 80.01 30.48)
 		)
@@
 	(wire
 		(pts
+			(xy 44.45 30.48) (xy 54.61 30.48)
+		)
+		(stroke
+			(width 0)
+			(type default)
+		)
+	)
+	(wire
+		(pts
 			(xy 101.6 30.48) (xy 106.68 30.48)
 		)
@@
 		(pts
 			(xy 104.14 38.1) (xy 104.14 39.37)
+		)
+		(stroke
+			(width 0)
+			(type default)
+		)
+	)
+	(wire
+		(pts
+			(xy 62.23 30.48) (xy 72.39 30.48)
 		)
 		(stroke
@@
 		)
 	)
-	(label "GND"
-		(at 67.31 33.02 0)
+	(label "5V_USB"
+		(at 44.45 30.48 0)
 		(effects
 			(font
@@
 	)
 	(symbol
-		(lib_id "Connector:Conn_01x02_Pin")
-		(at 62.23 30.48 0)
-		(unit 1)
-		(exclude_from_sim no)
-		(in_bom yes)
-		(on_board yes)
-		(dnp no)
-		(property "Reference" "J3"
-			(at 65.024 25.654 0)
-			(effects
-				(font
-					(size 0.7 0.7)
-				)
-			)
-		)
-		(property "Value" "Conn_01x02_Pin"
-			(at 65.024 26.924 0)
-			(effects
-				(font
-					(size 0.7 0.7)
-				)
-			)
-		)
-		(property "Footprint" ""
-			(at 62.23 30.48 0)
-			(effects
-				(font
-					(size 1.27 1.27)
-				)
-				(hide yes)
-			)
-		)
-		(property "Datasheet" "~"
-			(at 62.23 30.48 0)
-			(effects
-				(font
-					(size 1.27 1.27)
-				)
-				(hide yes)
-			)
-		)
-		(property "Description" "Generic connector, single row, 01x02, script generated"
-			(at 62.23 30.48 0)
-			(effects
-				(font
-					(size 1.27 1.27)
-				)
-				(hide yes)
-			)
-		)
-		(pin "2"
-		)
-		(pin "1"
-		)
-		(instances
-			(project ""
-				(path "/5559dfcd-b512-40eb-907e-1d8fde12bd30/cc3e6568-130d-4575-9c35-8244639d6b7b"
-					(reference "J3")
-					(unit 1)
-				)
-			)
-		)
-	)
-	(symbol
 		(lib_id "Device:C_Small")
 		(at 119.38 24.13 0)
@@
 	(symbol
 		(lib_id "Connector:USB_C_Receptacle_USB2.0_16P")
-		(at 29.21 39.37 0)
+		(at 29.21 45.72 0)
 		(unit 1)
 		(exclude_from_sim no)
@@
 		(fields_autoplaced yes)
 		(property "Reference" "J4"
-			(at 29.21 16.51 0)
+			(at 29.21 22.86 0)
 			(effects
 				(font
@@
 		)
 		(property "Value" "USB_C_Receptacle_USB2.0_16P"
-			(at 29.21 19.05 0)
+			(at 29.21 25.4 0)
 			(effects
 				(font
@@
 		)
 		(property "Footprint" ""
-			(at 33.02 39.37 0)
+			(at 33.02 45.72 0)
 			(effects
 				(font
@@
 		)
 		(property "Datasheet" "https://www.usb.org/sites/default/files/documents/usb_type-c.zip"
-			(at 33.02 39.37 0)
+			(at 33.02 45.72 0)
 			(effects
 				(font
@@
 		)
 		(property "Description" "USB 2.0-only 16P Type-C Receptacle connector"
-			(at 29.21 39.37 0)
+			(at 29.21 45.72 0)
 			(effects
 				(font
@@
 				(path "/5559dfcd-b512-40eb-907e-1d8fde12bd30/cc3e6568-130d-4575-9c35-8244639d6b7b"
 					(reference "J4")
-					(unit 1)
-				)
-			)
-		)
-	)
-	(symbol
-		(lib_id "power:PWR_FLAG")
-		(at 67.31 30.48 0)
-		(unit 1)
-		(exclude_from_sim no)
-		(in_bom yes)
-		(on_board yes)
-		(dnp no)
-		(fields_autoplaced yes)
-		(property "Reference" "#FLG08"
-			(at 67.31 28.575 0)
-			(effects
-				(font
-					(size 1.27 1.27)
-				)
-				(hide yes)
-			)
-		)
-		(property "Value" "PWR_FLAG"
-			(at 67.31 26.67 0)
-			(effects
-				(font
-					(size 0.7 0.7)
-				)
-				(hide yes)
-			)
-		)
-		(property "Footprint" ""
-			(at 67.31 30.48 0)
-			(effects
-				(font
-					(size 1.27 1.27)
-				)
-				(hide yes)
-			)
-		)
-		(property "Datasheet" "~"
-			(at 67.31 30.48 0)
-			(effects
-				(font
-					(size 1.27 1.27)
-				)
-				(hide yes)
-			)
-		)
-		(property "Description" "Special symbol for telling ERC where power comes from"
-			(at 67.31 30.48 0)
-			(effects
-				(font
-					(size 1.27 1.27)
-				)
-				(hide yes)
-			)
-		)
-		(pin "1"
-		)
-		(instances
-			(project ""
-				(path "/5559dfcd-b512-40eb-907e-1d8fde12bd30/cc3e6568-130d-4575-9c35-8244639d6b7b"
-					(reference "#FLG08")
 					(unit 1)
 				)
@@
 					(unit 1)
 				)
+			)
+		)
+	)
+	(symbol
+		(lib_id "Device:D_Schottky")
+		(at 58.42 30.48 0)
+		(unit 1)
+		(exclude_from_sim no)
+		(in_bom yes)
+		(on_board yes)
+		(dnp no)
+		(fields_autoplaced yes)
+		(property "Reference" "D2"
+			(at 58.1025 26.67 0)
+			(effects
+				(font
+					(size 0.7 0.7)
+				)
+			)
+		)
+		(property "Value" "D_Schottky"
+			(at 58.1025 27.94 0)
+			(effects
+				(font
+					(size 0.7 0.7)
+				)
+			)
+		)
+		(property "Footprint" ""
+			(at 58.42 30.48 0)
+			(effects
+				(font
+					(size 1.27 1.27)
+				)
+				(hide yes)
+			)
+		)
+		(property "Datasheet" "~"
+			(at 58.42 30.48 0)
+			(effects
+				(font
+					(size 1.27 1.27)
+				)
+				(hide yes)
+			)
+		)
+		(property "Description" "Schottky diode"
+			(at 58.42 30.48 0)
+			(effects
+				(font
+					(size 1.27 1.27)
+				)
+				(hide yes)
+			)
+		)
+		(pin "1"
+		)
+		(pin "2"
+		)
+		(instances
+			(project ""
+				(path "/5559dfcd-b512-40eb-907e-1d8fde12bd30/cc3e6568-130d-4575-9c35-8244639d6b7b"
+					(reference "D2")
+					(unit 1)
+				)
+			)
+		)
+	)
+	(symbol
+		(lib_id "Device:D_Schottky")
+		(at 58.42 40.64 0)
+		(unit 1)
+		(exclude_from_sim no)
+		(in_bom yes)
+		(on_board yes)
+		(dnp no)
+		(fields_autoplaced yes)
+		(property "Reference" "D3"
+			(at 58.1025 36.83 0)
+			(effects
+				(font
+					(size 0.7 0.7)
+				)
+			)
+		)
+		(property "Value" "D_Schottky"
+			(at 58.1025 38.1 0)
+			(effects
+				(font
+					(size 0.7 0.7)
+				)
+			)
+		)
+		(property "Footprint" ""
+			(at 58.42 40.64 0)
+			(effects
+				(font
+					(size 1.27 1.27)
+				)
+				(hide yes)
+			)
+		)
+		(property "Datasheet" "~"
+			(at 58.42 40.64 0)
+			(effects
+				(font
+					(size 1.27 1.27)
+				)
+				(hide yes)
+			)
+		)
+		(property "Description" "Schottky diode"
+			(at 58.42 40.64 0)
+			(effects
+				(font
+					(size 1.27 1.27)
+				)
+				(hide yes)
+			)
+		)
+		(pin "1"
+		)
+		(pin "2"
+		)
+		(instances
+			(project "SX1276"
+				(path "/5559dfcd-b512-40eb-907e-1d8fde12bd30/cc3e6568-130d-4575-9c35-8244639d6b7b"
+					(reference "D3")
+					(unit 1)
+				)

Commit message: until mcu
Parts:
- added C11: 10 µF, symbol Device:C_Small
- added C12: 100 nF, symbol Device:C_Small
- added J_BAT: Conn_01x02, symbol Connector_Generic:Conn_01x02
- added R1, R2: 5.1k, symbol Device:R_Small
- added U5: USBLC6-2SC6, Package_TO_SOT_SMD:SOT-23-6, symbol Power_Protection:USBLC6-2SC6
Connections:
- net +5V_IN is gone; now on net SYS_UPS: C3.2, D2.2 (A), U4.3 (VI)
- net 5V_USB: now also C11.1, C12.1
- net GND: now also C11.2, C12.2, J_BAT.2 (Pin_2), R1.2, R2.2, U5.2 (GND), U5.3 (I/O2)
- net at J4.A5 (CC1): now also R1.1
- net USB_DP: now reaches J4.A6 (D+)
- net USB_DP: now also J4.B6 (D+), U5.1 (I/O1)
- net USB_DM: now reaches J4.A7 (D-)
- net USB_DM: now also J4.B7 (D-), U5.5 (VBUS)
- net at J4.B5 (CC2): now also R2.1
- net BAT_RAW: now reaches D3.1 (K)
- net BAT_RAW: now also J_BAT.1 (Pin_1)
- net SYS_UPS: now reaches D3.2 (A)
- no-connect marks 0 -> 2
Other:
- note added: "CC pull-down"
- note removed: "Regülatör U4 - LM1117DT-3.3 Giriş: SYS_UPS (5-9 V arası) Çıkış: +3.3 V nominal Max Iout: ~800 mA Giriş/Çıkış farkı yüksek olduğunda termal kayıplar artar. Gerekirse buck regülatör alternatifi değerlendirilecektir."
- moved on the sheet: C3, C4, C5, C6, C7, D2, D3, FB3, U4
